Commit message: Fixed gear servo initial position

File: models/urdf/landing_rig.urdf (robot description, URDF)
Before this commit: robot uav_landing_rig, 4 links, 3 joints
Joints:
- joint landing_gear_joint: axis 1 0 0 -> -1 0 0

Commit message: Reworked kinematic joints

File: models/urdf/landing_rig.urdf (robot description, URDF)
Before this commit: robot uav_landing_rig, 4 links, 3 joints
Links:
- link base_link: geometry collision box size=0.16 0.16 0.04; visual box size=0.16 0.16 0.04
- link landing_gear_link: mass 0.05 -> 0.10; geometry collision cylinder length=0.18 radius=0.005; collision cylinder length=0.18 radius=0.005
- link sensor_plate_link: mass 0.08 -> 0.09; geometry collision cylinder length=0.006 radius=0.065; visual box size=0.010 0.012 0.003
Joints:
- joint fixed_mount: origin xyz=0 0 0.5 rpy=0 0 0 -> xyz=0 0 0.60 rpy=0 0 0
- joint landing_gear_joint: axis -1 0 0 -> 0 -1 0; limit lower=0.0 upper=1.5708 effort=1.0 velocity=4.0 -> lower=0.0 upper=1.5708 effort=1.5 velocity=4.0; origin xyz=0.0 0.0 -0.025 rpy=0 0 0 -> xyz=-0.04 0.0 -0.02 rpy=0 0 0
- joint pitch_stabilizer_joint: origin xyz=0.0 0.0 -0.035 rpy=0 0 0 -> xyz=0.04 0.0 -0.035 rpy=0 0 0

Commit message: Updated aircraft geometry to resemble a fixed wing airfract. Created t-tail

File: models/urdf/landing_rig.urdf (robot description, URDF)
Before this commit: robot uav_landing_rig, 4 links, 3 joints
Links:
- removed link sensor_plate_link
- added link horizontal_stabilizer_link, mass 0.05; collision box size=0.08 0.36 0.008; visual box size=0.08 0.36 0.008
- link base_link: mass 1.20 -> 1.60; geometry collision box size=0.11 0.014 0.16; collision box size=0.16 0.90 0.015
- link landing_gear_link: mass 0.10 -> 0.11; geometry collision cylinder length=0.016 radius=0.024; collision cylinder length=0.016 radius=0.024
Joints:
- removed joint pitch_stabilizer_joint
- added joint horizontal_stabilizer_joint: type revolute, parent base_link, child horizontal_stabilizer_link, origin xyz=-0.335 0 0.21 rpy=0 0 0, axis 0 1 0, limit lower=-0.4363 upper=0.4363 effort=1.2 velocity=6.0
- joint fixed_mount: origin xyz=0 0 0.60 rpy=0 0 0 -> xyz=0 0 0.70 rpy=0 0 0
- joint landing_gear_joint: limit lower=0.0 upper=1.5708 effort=1.5 velocity=4.0 -> lower=0.0 upper=1.5708 effort=2.0 velocity=3.5; origin xyz=-0.04 0.0 -0.02 rpy=0 0 0 -> xyz=0.04 0 -0.05 rpy=0 0 0

Commit message: Debugging active gear conditional control

File: models/urdf/landing_rig.urdf (robot description, URDF)
Before this commit: robot uav_landing_rig, 4 links, 3 joints
Links:
- added link flight_x_carriage, mass 0.01
Joints:
- removed joint fixed_mount
- added joint flight_x_joint: type prismatic, parent world, child flight_x_carriage, origin xyz=0 0 0 rpy=0 0 0, axis 1 0 0, limit lower=-5.0 upper=120.0 effort=500.0 velocity=10.0
- added joint flight_z_joint: type prismatic, parent flight_x_carriage, child base_link, origin xyz=0 0 0 rpy=0 0 0, axis 0 0 1, limit lower=0.0 upper=5.0 effort=500.0 velocity=5.0

Commit message: Still debugging landing problem

File: models/urdf/landing_rig.urdf (robot description, URDF)
Before this commit: robot uav_landing_rig, 5 links, 4 joints
Joints:
- joint flight_z_joint: limit lower=0.0 upper=5.0 effort=500.0 velocity=5.0 -> lower=0.10 upper=3.0 effort=500.0 velocity=5.0
